Commit message: robotfun_description: brazo 4 GDL, esqueleto único (medidas reales + piezas reales)
- urdf/common/arm.macro.xacro: esqueleto compartido con los orígenes REALES de
  brazo_ws y los pitch en axis="0 -1 0" → reproduce EXACTAMENTE la FK del núcleo
  (TF==FK a 1e-16). Param use_mesh selecciona primitivas o meshes.
- robotfun.urdf.xacro: MEDIDAS REALES (primitivas) — para verificar la IK.
- robotfun_meshes.urdf.xacro: PIEZAS REALES (meshes del CAD, ya limpias) + gripper
  real de twin_ws. Misma interfaz de juntas que el primitivo → mismo /joint_states.
- Limpieza: eliminado eslabon3_1link.stl (pieza sobrante); corregida la escala de
  eslabon3 (0.001 → 0.0001; a 0.001 flotaba a ~2.4 m).
- scripts/verify_kinematics.py (sustituye generate_dh_origins): prueba la
  equivalencia esqueleto↔DH. mesh_bbox.py actualizado para guiar el centrado.
- config/joint_limits, initial_positions a 4 GDL.

Co-Authored-By: Claude Opus 4.8 <noreply@anthropic.com>
Claude-Session: https://claude.ai/code/session_01HQm53DmrqYUT2G9sJ8qfUh

File: src/robotfun_description/urdf/robotfun.urdf.xacro (robot description, xacro)
@@ -1,172 +1,18 @@
 <?xml version="1.0"?>
 <!-- ============================================================================
-     robotfun.urdf.xacro  —  MODELO CANÓNICO (primitivas, DH-exacto)
+     robotfun.urdf.xacro  —  MODELO DE MEDIDAS REALES (primitivas)
      ===========================================================================
-     Brazo de 5 GDL (RRRRR) + gripper, generado DIRECTAMENTE desde la tabla DH
-     **validada** de `robotfun_kinematics.core.dh_model`. Los orígenes de los
-     joints provienen de `scripts/generate_dh_origins.py`, que verifica TF == FK
-     a 1e-12 (FK(HOME) = [0.010, 0, 0.393] m).
-         L0=0.010 L1=0.063 L2=0.120 L3=0.090 L4=0.030 L5=0.090 (m)
-     Este es el modelo de referencia para cinemática, MoveIt2 y Gazebo (incluye
-     <collision> e <inertial>). Para comparar con las piezas reales del robot,
-     usar el modelo de meshes:  display.launch.py model:=meshes
+     Brazo 4 GDL (yaw + 3 pitch) + gripper, dibujado con PRIMITIVAS dimensionadas
+     a las medidas reales del robot. Comparte el esqueleto (juntas joint_1..joint_4)
+     con el modelo de meshes, y reproduce EXACTAMENTE la FK del núcleo
+     `robotfun_kinematics` (TF == FK). Es el modelo para VERIFICAR la cinemática
+     inversa. Incluye inertiales (preparado para Gazebo/MoveIt2).
+     Para ver las piezas reales del CAD:  display.launch.py model:=meshes
      ========================================================================== -->
 <robot name="robotfun" xmlns:xacro="http://www.ros.org/wiki/xacro">
   <xacro:include filename="$(find robotfun_description)/urdf/common/materials.xacro"/>
+  <xacro:include filename="$(find robotfun_description)/urdf/common/arm.macro.xacro"/>
   <xacro:include filename="$(find robotfun_description)/urdf/common/gripper.macro.xacro"/>
-  <xacro:property name="L1" value="0.063"/>
-  <xacro:property name="L2" value="0.120"/>
-  <xacro:property name="L4_len" value="0.120"/>  <!-- L3+L4 -->
-  <xacro:property name="L5" value="0.090"/>
-  <xacro:property name="lower" value="-1.5708"/> <!-- ±90°, igual que el firmware -->
-  <xacro:property name="upper" value="1.5708"/>
-  <!-- ===================== mundo / base ===================== -->
-  <link name="world"/>
-  <link name="base_link">
-    <inertial>
-      <mass value="1.0"/>
-      <inertia ixx="0.01" ixy="0" ixz="0" iyy="0.01" iyz="0" izz="0.01"/>
-    </inertial>
-    <visual>
-      <origin xyz="0 0 -0.015" rpy="0 0 0"/>
-      <geometry><cylinder radius="0.05" length="0.03"/></geometry>
-      <material name="grey"/>
-    </visual>
-    <collision>
-      <origin xyz="0 0 -0.015" rpy="0 0 0"/>
-      <geometry><cylinder radius="0.05" length="0.03"/></geometry>
-    </collision>
-  </link>
-  <joint name="base_joint" type="fixed">
-    <origin xyz="0 0 0" rpy="0 0 0"/>
-    <parent link="world"/><child link="base_link"/>
-  </joint>
-  <!-- ===================== link_1 (J1 yaw base) ===================== -->
-  <link name="link_1">
-    <inertial>
-      <origin xyz="0 0 0.0315" rpy="0 0 0"/><mass value="0.5"/>
-      <inertia ixx="1e-3" ixy="0" ixz="0" iyy="1e-3" iyz="0" izz="1e-3"/>
-    </inertial>
-    <visual>
-      <origin xyz="0 0 0.0315" rpy="0 0 0"/>
-      <geometry><cylinder radius="0.018" length="${L1}"/></geometry>
-      <material name="black"/>
-    </visual>
-    <collision>
-      <origin xyz="0 0 0.0315" rpy="0 0 0"/>
-      <geometry><cylinder radius="0.018" length="${L1}"/></geometry>
-    </collision>
-  </link>
-  <joint name="joint_1" type="revolute">
-    <origin xyz="0.000000 0.000000 0.000000" rpy="0.000000 0.000000 0.000000"/>
-    <parent link="base_link"/><child link="link_1"/>
-    <axis xyz="0 0 1"/>
-    <limit effort="30.0" lower="${lower}" upper="${upper}" velocity="3.0"/>
-  </joint>
-  <!-- ===================== link_2 (J2 hombro, a2=L2) ===================== -->
-  <link name="link_2">
-    <inertial>
-      <origin xyz="0.06 0 0" rpy="0 0 0"/><mass value="0.5"/>
-      <inertia ixx="1e-3" ixy="0" ixz="0" iyy="1e-3" iyz="0" izz="1e-3"/>
-    </inertial>
-    <visual>
-      <origin xyz="0.060 0 0" rpy="0 1.570796 0"/>
-      <geometry><cylinder radius="0.016" length="${L2}"/></geometry>
-      <material name="red"/>
-    </visual>
-    <collision>
-      <origin xyz="0.060 0 0" rpy="0 1.570796 0"/>
-      <geometry><cylinder radius="0.016" length="${L2}"/></geometry>
-    </collision>
-  </link>
-  <joint name="joint_2" type="revolute">
-    <origin xyz="0.010000 0.000000 0.063000" rpy="1.570796 -1.570796 0.000000"/>
-    <parent link="link_1"/><child link="link_2"/>
-    <axis xyz="0 0 1"/>
-    <limit effort="30.0" lower="${lower}" upper="${upper}" velocity="3.0"/>
-  </joint>
-  <!-- ===================== link_3 (J3 codo, Z3 colineal → nodo) ===== -->
-  <link name="link_3">
-    <inertial>
-      <mass value="0.2"/>
-      <inertia ixx="5e-4" ixy="0" ixz="0" iyy="5e-4" iyz="0" izz="5e-4"/>
-    </inertial>
-    <visual>
-      <origin xyz="0 0 0" rpy="0 0 0"/>
-      <geometry><sphere radius="0.020"/></geometry>
-      <material name="black"/>
-    </visual>
-    <collision>
-      <origin xyz="0 0 0" rpy="0 0 0"/>
-      <geometry><sphere radius="0.020"/></geometry>
-    </collision>
-  </link>
-  <joint name="joint_3" type="revolute">
-    <origin xyz="0.120000 0.000000 0.000000" rpy="0.000000 0.000000 1.570796"/>
-    <parent link="link_2"/><child link="link_3"/>
-    <axis xyz="0 0 1"/>
-    <limit effort="30.0" lower="${lower}" upper="${upper}" velocity="3.0"/>
-  </joint>
-  <!-- ===================== link_4 (J4 ROLL antebrazo, d4=L3+L4) ===== -->
-  <link name="link_4">
-    <inertial>
-      <origin xyz="0 0 0.06" rpy="0 0 0"/><mass value="0.3"/>
-      <inertia ixx="8e-4" ixy="0" ixz="0" iyy="8e-4" iyz="0" izz="8e-4"/>
-    </inertial>
-    <visual>
-      <origin xyz="0 0 0.060" rpy="0 0 0"/>
-      <geometry><cylinder radius="0.014" length="${L4_len}"/></geometry>
-      <material name="blue"/>
-    </visual>
-    <collision>
-      <origin xyz="0 0 0.060" rpy="0 0 0"/>
-      <geometry><cylinder radius="0.014" length="${L4_len}"/></geometry>
-    </collision>
-  </link>
-  <joint name="joint_4" type="revolute">
-    <origin xyz="0.000000 0.000000 0.000000" rpy="1.570796 0.000000 0.000000"/>
-    <parent link="link_3"/><child link="link_4"/>
-    <axis xyz="0 0 1"/>
-    <limit effort="30.0" lower="${lower}" upper="${upper}" velocity="3.0"/>
-  </joint>
-  <!-- ===================== link_5 (J5 muñeca pitch, a5=L5) ========== -->
-  <link name="link_5">
-    <inertial>
-      <origin xyz="0.045 0 0" rpy="0 0 0"/><mass value="0.2"/>
-      <inertia ixx="5e-4" ixy="0" ixz="0" iyy="5e-4" iyz="0" izz="5e-4"/>
-    </inertial>
-    <visual>
-      <origin xyz="0.045 0 0" rpy="0 1.570796 0"/>
-      <geometry><cylinder radius="0.013" length="${L5}"/></geometry>
-      <material name="black"/>
-    </visual>
-    <collision>
-      <origin xyz="0.045 0 0" rpy="0 1.570796 0"/>
-      <geometry><cylinder radius="0.013" length="${L5}"/></geometry>
-    </collision>
-  </link>
-  <joint name="joint_5" type="revolute">
-    <origin xyz="0.000000 0.000000 0.120000" rpy="1.570796 -1.570796 0.000000"/>
-    <parent link="link_4"/><child link="link_5"/>
-    <axis xyz="0 0 1"/>
-    <limit effort="30.0" lower="${lower}" upper="${upper}" velocity="3.0"/>
-  </joint>
-  <!-- ===================== efector final (tool0) ===================== -->
-  <link name="tool0">
-    <inertial>
-      <mass value="0.05"/>
-      <inertia ixx="1e-4" ixy="0" ixz="0" iyy="1e-4" iyz="0" izz="1e-4"/>
-    </inertial>
-    <visual>
-      <origin xyz="0 0 0" rpy="0 0 0"/>
-      <geometry><box size="0.02 0.03 0.012"/></geometry>
-      <material name="grey"/>
-    </visual>
-  </link>
-  <joint name="tool_fixed" type="fixed">
-    <origin xyz="0.090000 0.000000 0.000000" rpy="0.000000 0.000000 0.000000"/>
-    <parent link="link_5"/><child link="tool0"/>
-  </joint>
-  <!-- ===================== gripper (canal 6, primitivo) ============== -->
+  <xacro:robotfun_arm use_mesh="false"/>
   <xacro:gripper_primitive parent="tool0">
     <origin xyz="0 0 0.006" rpy="0 0 0"/>

File: src/robotfun_description/urdf/robotfun_meshes.urdf.xacro (robot description, xacro)
@@ -1,119 +1,26 @@
 <?xml version="1.0"?>
 <!-- ============================================================================
-     robotfun_meshes.urdf.xacro  —  MODELO DE MESHES REALES (reparado)
+     robotfun_meshes.urdf.xacro  —  MODELO DE PIEZAS REALES (meshes del CAD)
      ===========================================================================
-     Reparación del `brazo.urdf` original (brazo_ws) para visualizar las piezas
-     CAD reales del robot y COMPARARLAS con el modelo canónico de primitivas
-     (`robotfun.urdf.xacro`). Comparten la MISMA interfaz de juntas
-     (joint_1..joint_5 + gripper), por lo que el mismo /joint_states mueve ambos.
-     Correcciones aplicadas frente al brazo.urdf original:
-       * Juntas renombradas joint1..joint5 → joint_1..joint_5 (consistencia con
-         el núcleo de cinemática y el firmware).
-       * Eliminados engranaje1/2_link y sus joints: referenciaban
-         Engranaje1.stl / Engranaje2.stl INEXISTENTES (rompían la carga) y usaban
-         rpy en GRADOS (URDF usa radianes). En su lugar se monta el gripper real
-         rescatado de twin_ws.
-       * Límites articulares saturados a ±90° (±1.5708), coherente con los servos
-         físicos y con el firmware.
-       * Meshes referenciadas desde robotfun_description/meshes/arm.
-     CENTRADO (pendiente de afinar en TU RViz): las STL están en un marco CAD
-     global común; el `<origin>` de cada <visual> solo compensa Z. Ejecuta
-     `scripts/mesh_bbox.py` y ajusta XY, o re-exporta los STL re-origenados.
-     El modelo PRIMITIVO es la referencia cinemática correcta (TF == FK).
+     Mismo esqueleto y MISMAS juntas (joint_1..joint_4) que el modelo de medidas
+     reales, pero con las PIEZAS REALES del robot (meshes de brazo_ws, ya limpio:
+     sin engranajes ni eslabón sobrante, escala uniforme 0.001). Sirve para ver
+     el robot tal cual es y comparar con el modelo primitivo (ambos se mueven
+     idéntico, los mueve el mismo /joint_states). Se monta el GRIPPER real
+     rescatado de twin_ws.
+     CENTRADO de meshes: las STL vienen en un marco CAD global; el <visual> de
+     cada link compensa la traslación. Si alguna pieza se ve descentrada en XY,
+     ajusta su <origin> (ver scripts/mesh_bbox.py). El modelo primitivo es la
+     referencia cinemática exacta.
      ========================================================================== -->
 <robot name="robotfun_meshes" xmlns:xacro="http://www.ros.org/wiki/xacro">
   <xacro:include filename="$(find robotfun_description)/urdf/common/materials.xacro"/>
+  <xacro:include filename="$(find robotfun_description)/urdf/common/arm.macro.xacro"/>
   <xacro:include filename="$(find robotfun_description)/urdf/common/gripper.macro.xacro"/>
-  <xacro:property name="lower" value="-1.5708"/>
-  <xacro:property name="upper" value="1.5708"/>
-  <xacro:property name="mesh" value="package://robotfun_description/meshes/arm"/>
-  <!-- mundo / base (raíz 'world' igual que el modelo primitivo) -->
-  <link name="world"/>
-  <joint name="base_joint" type="fixed">
-    <origin xyz="0 0 0" rpy="0 0 0"/>
-    <parent link="world"/><child link="base_link"/>
-  </joint>
-  <link name="base_link">
-    <inertial>
-      <mass value="1.0"/>
-      <inertia ixx="0.01" ixy="0" ixz="0" iyy="0.01" iyz="0" izz="0.01"/>
-    </inertial>
-    <visual>
-      <origin xyz="0.0 0.0 0.0" rpy="0.0 0.0 0.0"/>
-      <geometry><mesh filename="${mesh}/base_link.stl" scale="0.001 0.001 0.001"/></geometry>
-      <material name="black"/>
-    </visual>
-  </link>
-  <link name="eslabon1_link">
-    <visual>
-      <origin xyz="0.0 0.0 -0.0617" rpy="0.0 0.0 0.0"/>
-      <geometry><mesh filename="${mesh}/eslabon1_link.stl" scale="0.001 0.001 0.001"/></geometry>
-      <material name="white_grey"/>
-    </visual>
-  </link>
-  <joint name="joint_1" type="revolute">
-    <parent link="base_link"/><child link="eslabon1_link"/>
-    <origin xyz="0.0 0.0 0.0617" rpy="0.0 0.0 0.0"/>
-    <axis xyz="0 0 1"/>
-    <limit lower="${lower}" upper="${upper}" effort="10.0" velocity="1.0"/>
-  </joint>
-  <link name="eslabon2_link">
-    <visual>
-      <origin xyz="0.0 0.0 -0.1375" rpy="0.0 0.0 0.0"/>
-      <geometry><mesh filename="${mesh}/eslabon2_link.stl" scale="0.001 0.001 0.001"/></geometry>
-      <material name="white_grey"/>
-    </visual>
-  </link>
-  <joint name="joint_2" type="revolute">
-    <parent link="eslabon1_link"/><child link="eslabon2_link"/>
-    <origin xyz="0.0 0.0 0.0758" rpy="0.0 0.0 0.0"/>
-    <axis xyz="0 1 0"/>
-    <limit lower="${lower}" upper="${upper}" effort="10.0" velocity="1.0"/>
-  </joint>
-  <!-- eslabon3 / eslabon3_1: escala 0.0001 (exportados 10x); ver mesh_bbox.py -->
-  <link name="eslabon3_link">
-    <visual>
-      <origin xyz="0.0 0.0 -0.2652" rpy="0.0 0.0 0.0"/>
-      <geometry><mesh filename="${mesh}/eslabon3_link.stl" scale="0.0001 0.0001 0.0001"/></geometry>
-      <material name="white_grey"/>
-    </visual>
-  </link>
-  <joint name="joint_3" type="revolute">
-    <parent link="eslabon2_link"/><child link="eslabon3_link"/>
-    <origin xyz="0.0 0.0 0.1277" rpy="0.0 0.0 0.0"/>
-    <axis xyz="0 1 0"/>
-    <limit lower="${lower}" upper="${upper}" effort="10.0" velocity="1.0"/>
-  </joint>
-  <link name="eslabon3_1link">
-    <visual>
-      <origin xyz="0.0 0.0 -0.2652" rpy="0.0 0.0 0.0"/>
-      <geometry><mesh filename="${mesh}/eslabon3_1link.stl" scale="0.0001 0.0001 0.0001"/></geometry>
-      <material name="white_grey"/>
-    </visual>
-  </link>
-  <joint name="joint_4" type="revolute">
-    <parent link="eslabon3_link"/><child link="eslabon3_1link"/>
-    <origin xyz="0.00140 0.0 0.00140" rpy="0.0 0.0 0.0"/>
-    <axis xyz="0 0 1"/>
-    <limit lower="${lower}" upper="${upper}" effort="10.0" velocity="1.0"/>
-  </joint>
-  <link name="eslabon4_link">
-    <visual>
-      <origin xyz="-0.038 0.0 -0.3865" rpy="0.0 0.0 0.0"/>
-      <geometry><mesh filename="${mesh}/eslabon4_link.stl" scale="0.001 0.001 0.001"/></geometry>
-      <material name="black"/>
-    </visual>
-  </link>
-  <joint name="joint_5" type="revolute">
-    <parent link="eslabon3_1link"/><child link="eslabon4_link"/>
-    <origin xyz="0.038 0.0 0.1213" rpy="0.0 0.0 0.0"/>
-    <axis xyz="0 1 0"/>
-    <limit lower="${lower}" upper="${upper}" effort="10.0" velocity="1.0"/>
-  </joint>
-  <!-- ============ gripper real rescatado de twin_ws (canal 6) ============ -->
-  <!-- Sustituye los engranajes inexistentes del brazo.urdf original. El offset
-       de placement es un punto de partida: afínalo en RViz (ver README). -->
-  <xacro:gripper_mesh parent="eslabon4_link" grip_z="-0.40">
-    <origin xyz="0.038 0.0 0.1213" rpy="0 0 0"/>
+  <xacro:robotfun_arm use_mesh="true"/>
+  <!-- Gripper real (twin_ws) en el TCP. El offset es punto de partida: afínalo
+       en RViz si hace falta (ver README). -->
+  <xacro:gripper_mesh parent="tool0" grip_z="-0.03">
+    <origin xyz="0 0 0.0" rpy="0 0 0"/>
   </xacro:gripper_mesh>
 </robot>
