Commit message: 4 GDL: brazo recto con medidas reales, gripper fusionado y sin cubo
Cambios pedidos por el usuario (con sus medidas reales):
- Medidas: antebrazo A3=0.125 m y mano HAND=0.12 m (medidas del usuario). Se
  adopta un brazo RECTO (sin el offset de 17°): DH más limpia y verificable.
  FK(HOME) → TCP=[0,0,0.5102]; TF==FK a 1e-16 (verify_kinematics.py).
- Restricción articular literal −90/0/+90 (HOME=0 ⇒ servo a 90°): es la que ya
  estaba; se confirma en límites del URDF y del núcleo.
- URDF de hardware (model:=meshes): tool0 deja de tener cubo (solo frame); el
  gripper real (twin_ws) se FUSIONA a link_4 como un solo cuerpo rígido
  (gripper_mesh_fused), sin piezas flotando. Mallas re-centradas al esqueleto
  recto. El modelo primitivo usa un gripper de dedos finos (sin cubo).
- Núcleo/tests/docs actualizados a las medidas y al modelo recto.

Ambos modelos (medidas reales / piezas reales) comparten juntas joint_1..joint_4
y se mueven con el mismo /joint_states.

Co-Authored-By: Claude Opus 4.8 <noreply@anthropic.com>
Claude-Session: https://claude.ai/code/session_01HQm53DmrqYUT2G9sJ8qfUh

File: src/robotfun_description/urdf/common/arm.macro.xacro (robot description, xacro)
@@ -1,20 +1,19 @@
 <?xml version="1.0"?>
 <!-- ============================================================================
-     arm.macro.xacro  —  esqueleto compartido del brazo 4 GDL
+     arm.macro.xacro  —  esqueleto compartido del brazo 4 GDL (RECTO)
      ===========================================================================
-     Define la cadena cinemática (base_link → link_1..link_4 → tool0) con los
-     orígenes REALES del robot (brazo_ws) y los ejes corregidos para que el URDF
-     reproduzca EXACTAMENTE la FK del núcleo `robotfun_kinematics` (verificado a
-     0.0). El mismo esqueleto sirve para los dos modelos:
-        use_mesh=false → visual con PRIMITIVAS dimensionadas a las medidas reales.
-        use_mesh=true  → visual con las PIEZAS REALES del CAD (meshes).
-     Así ambos modelos comparten juntas (joint_1..joint_4) y se mueven idénticos.
-     Ejes: joint_1 = (0 0 1) [yaw]; joint_2/3/4 = (0 -1 0) [pitch]. El signo −1
-     en los pitch es lo que hace coincidir el giro con la convención DH del núcleo.
+     Cadena base_link → link_1..link_4 → tool0 con las medidas reales y el brazo
+     RECTO (sin offsets). Reproduce EXACTAMENTE la FK del núcleo (TF == FK a 1e-16).
+         D1=0.1375  A2=0.1277  A3=0.125 (medido)  HAND=0.12 (medido)  [m]
+     El mismo esqueleto sirve para los dos modelos:
+        use_mesh=false → PRIMITIVAS dimensionadas a las medidas (verifica DH/IK).
+        use_mesh=true  → PIEZAS REALES del CAD (visualización del hardware).
+     Ejes: joint_1=(0 0 1) yaw; joint_2/3/4=(0 -1 0) pitch. tool0 es solo un frame
+     (sin cubo). El gripper se añade aparte (gripper.macro.xacro).
      ========================================================================== -->
 <robot xmlns:xacro="http://www.ros.org/wiki/xacro">
   <xacro:property name="mesh" value="package://robotfun_description/meshes/arm"/>
-  <xacro:property name="lo" value="-1.5708"/>   <!-- ±90°, igual que los servos -->
-  <xacro:property name="hi" value="1.5708"/>
+  <xacro:property name="lo" value="-1.5708"/>   <!-- −90°, límite real del servo -->
+  <xacro:property name="hi" value="1.5708"/>    <!-- +90° (HOME=0 ⇒ servo a 90°) -->
   <xacro:macro name="robotfun_arm" params="use_mesh:=false">
     <link name="world"/>
@@ -41,6 +40,5 @@
     <joint name="joint_1" type="revolute">
       <origin xyz="0 0 0.0617" rpy="0 0 0"/><parent link="base_link"/><child link="link_1"/>
-      <axis xyz="0 0 1"/>
-      <limit lower="${lo}" upper="${hi}" effort="10.0" velocity="1.5"/>
+      <axis xyz="0 0 1"/><limit lower="${lo}" upper="${hi}" effort="10.0" velocity="1.5"/>
     </joint>
     <!-- ===== link_1 (yaw → hombro) ===== -->
@@ -63,8 +61,7 @@
     <joint name="joint_2" type="revolute">
       <origin xyz="0 0 0.0758" rpy="0 0 0"/><parent link="link_1"/><child link="link_2"/>
-      <axis xyz="0 -1 0"/>
-      <limit lower="${lo}" upper="${hi}" effort="10.0" velocity="1.5"/>
+      <axis xyz="0 -1 0"/><limit lower="${lo}" upper="${hi}" effort="10.0" velocity="1.5"/>
     </joint>
-    <!-- ===== link_2 (brazo) ===== -->
+    <!-- ===== link_2 (brazo, A2) ===== -->
     <link name="link_2">
       <inertial><origin xyz="0 0 0.064"/><mass value="0.4"/>
@@ -85,15 +82,13 @@
     <joint name="joint_3" type="revolute">
       <origin xyz="0 0 0.1277" rpy="0 0 0"/><parent link="link_2"/><child link="link_3"/>
-      <axis xyz="0 -1 0"/>
-      <limit lower="${lo}" upper="${hi}" effort="10.0" velocity="1.5"/>
+      <axis xyz="0 -1 0"/><limit lower="${lo}" upper="${hi}" effort="10.0" velocity="1.5"/>
     </joint>
-    <!-- ===== link_3 (antebrazo, con el offset radial real 0.038) ===== -->
+    <!-- ===== link_3 (antebrazo, A3=0.125) ===== -->
     <link name="link_3">
-      <inertial><origin xyz="0.019 0 0.061"/><mass value="0.3"/>
+      <inertial><origin xyz="0 0 0.0625"/><mass value="0.3"/>
         <inertia ixx="8e-4" ixy="0" ixz="0" iyy="8e-4" iyz="0" izz="8e-4"/></inertial>
       <visual>
         <xacro:if value="${use_mesh}">
-          <!-- eslabon3 se exportó en otro marco/escala: usa 0.0001 (a 0.001 flota
-               a ~2.4 m). Su centrado XY puede requerir ajuste fino en RViz. -->
+          <!-- eslabon3 se exportó en otra escala: usa 0.0001 (a 0.001 flota a ~2.4 m). -->
           <origin xyz="0 0 -0.2652" rpy="0 0 0"/>
           <geometry><mesh filename="${mesh}/eslabon3_link.stl" scale="0.0001 0.0001 0.0001"/></geometry>
@@ -101,6 +96,6 @@
         </xacro:if>
         <xacro:unless value="${use_mesh}">
-          <origin xyz="0.019 0 0.0607" rpy="0 0.3036 0"/>
-          <geometry><cylinder radius="0.015" length="0.1271"/></geometry>
+          <origin xyz="0 0 0.0625" rpy="0 0 0"/>
+          <geometry><cylinder radius="0.015" length="0.125"/></geometry>
           <material name="blue"/>
         </xacro:unless>
@@ -108,38 +103,31 @@
     </link>
     <joint name="joint_4" type="revolute">
-      <origin xyz="0.038 0 0.1213" rpy="0 0 0"/><parent link="link_3"/><child link="link_4"/>
-      <axis xyz="0 -1 0"/>
-      <limit lower="${lo}" upper="${hi}" effort="10.0" velocity="1.5"/>
+      <origin xyz="0 0 0.125" rpy="0 0 0"/><parent link="link_3"/><child link="link_4"/>
+      <axis xyz="0 -1 0"/><limit lower="${lo}" upper="${hi}" effort="10.0" velocity="1.5"/>
     </joint>
-    <!-- ===== link_4 (muñeca → mano) ===== -->
+    <!-- ===== link_4 (muñeca + base del gripper = UN solo eslabón) =====
+         En el modelo de meshes, link_4 = eslabon4 (pieza de muñeca/soporte del
+         gripper). El gripper se fusiona aquí mismo (gripper.macro.xacro). -->
     <link name="link_4">
-      <inertial><origin xyz="0 0 0.05"/><mass value="0.15"/>
+      <inertial><origin xyz="0 0 0.06"/><mass value="0.2"/>
         <inertia ixx="5e-4" ixy="0" ixz="0" iyy="5e-4" iyz="0" izz="5e-4"/></inertial>
       <visual>
         <xacro:if value="${use_mesh}">
-          <origin xyz="-0.038 0 -0.3865" rpy="0 0 0"/>
+          <origin xyz="0 0 -0.3902" rpy="0 0 0"/>
           <geometry><mesh filename="${mesh}/eslabon4_link.stl" scale="0.001 0.001 0.001"/></geometry>
           <material name="black"/>
         </xacro:if>
         <xacro:unless value="${use_mesh}">
-          <origin xyz="0 0 0.05" rpy="0 0 0"/>
-          <geometry><cylinder radius="0.013" length="0.10"/></geometry>
+          <origin xyz="0 0 0.06" rpy="0 0 0"/>
+          <geometry><cylinder radius="0.013" length="0.12"/></geometry>
           <material name="black"/>
         </xacro:unless>
       </visual>
     </link>
-    <!-- ===== tool0 (TCP, HAND=0.10 sobre la muñeca) ===== -->
+    <!-- tool0 = TCP (punta del gripper, HAND=0.12). Solo FRAME, sin cubo. -->
     <joint name="tool_fixed" type="fixed">
-      <origin xyz="0 0 0.10" rpy="0 0 0"/><parent link="link_4"/><child link="tool0"/>
+      <origin xyz="0 0 0.12" rpy="0 0 0"/><parent link="link_4"/><child link="tool0"/>
     </joint>
-    <link name="tool0">
-      <inertial><mass value="0.03"/>
-        <inertia ixx="1e-4" ixy="0" ixz="0" iyy="1e-4" iyz="0" izz="1e-4"/></inertial>
-      <visual>
-        <origin xyz="0 0 0" rpy="0 0 0"/>
-        <geometry><box size="0.03 0.04 0.012"/></geometry>
-        <material name="grey"/>
-      </visual>
-    </link>
+    <link name="tool0"/>
   </xacro:macro>
 </robot>

File: src/robotfun_description/urdf/common/gripper.macro.xacro (robot description, xacro)
@@ -2,89 +2,56 @@
 <!-- ============================================================================
      gripper.macro.xacro
-     Gripper de 1 GDL (canal 6). El servo `gripper` abre/cierra: un dedo es
-     accionado (joint "gripper") y el opuesto lo sigue con <mimic multiplier="-1">.
-     Esto reproduce en /joint_states y /joint_command el 6º valor [.. , gripper].
-     Dos macros (sin condicionales internos, más legibles):
-       * gripper_primitive : dedos de caja (modelo canónico / primitivo).
-       * gripper_mesh      : dedos con los STL reales rescatados de twin_ws.
-     El gripper real está en marco global (como las demás meshes): el offset de
-     placement es un punto de partida y se afina en RViz (ver README).
+     Dos macros, sin el cubo anterior:
+       * gripper_primitive : gripper de 1 GDL (canal 6) con dedos finos de caja;
+         se mueve (joint "gripper") para el modelo de medidas reales.
+       * gripper_mesh_fused: el gripper real (STL de twin_ws) FUSIONADO y FIJO al
+         eslabón de la muñeca → "un solo eslabón" con link_4. Sin cubo, sin flotar.
      ========================================================================== -->
 <robot xmlns:xacro="http://www.ros.org/wiki/xacro">
-  <!-- ===== PRIMITIVO ===== -->
+  <!-- ===== PRIMITIVO (móvil) ===== -->
   <xacro:macro name="gripper_primitive" params="parent *origin">
-    <link name="gripper_base">
-      <inertial>
-        <mass value="0.03"/>
-        <inertia ixx="1e-5" ixy="0" ixz="0" iyy="1e-5" iyz="0" izz="1e-5"/>
-      </inertial>
+    <joint name="gripper" type="revolute">
+      <xacro:insert_block name="origin"/>
+      <parent link="${parent}"/><child link="gripper_finger_left"/>
+      <axis xyz="0 1 0"/>
+      <limit effort="5.0" lower="0.0" upper="0.6" velocity="2.0"/>
+    </joint>
+    <link name="gripper_finger_left">
+      <inertial><mass value="0.01"/>
+        <inertia ixx="1e-6" ixy="0" ixz="0" iyy="1e-6" iyz="0" izz="1e-6"/></inertial>
       <visual>
-        <origin xyz="0 0 0.005" rpy="0 0 0"/>
-        <geometry><box size="0.03 0.05 0.01"/></geometry>
-        <material name="grey"/>
+        <origin xyz="0.012 0 0.018" rpy="0 0 0"/>
+        <geometry><box size="0.006 0.012 0.036"/></geometry>
+        <material name="red"/>
       </visual>
-      <collision>
-        <origin xyz="0 0 0.005" rpy="0 0 0"/>
-        <geometry><box size="0.03 0.05 0.01"/></geometry>
-      </collision>
     </link>
-    <joint name="gripper_mount" type="fixed">
+    <joint name="gripper_right" type="revolute">
       <xacro:insert_block name="origin"/>
-      <parent link="${parent}"/>
-      <child link="gripper_base"/>
-    </joint>
-    <xacro:gripper_finger_primitive side="left"  reflect="1"/>
-    <xacro:gripper_finger_primitive side="right" reflect="-1"/>
-    <!-- dedo accionado (left) -->
-    <joint name="gripper" type="revolute">
-      <origin xyz="0.0 0.018 0.01" rpy="0 0 0"/>
-      <parent link="gripper_base"/>
-      <child link="gripper_finger_left"/>
-      <axis xyz="1 0 0"/>
-      <limit effort="5.0" lower="0.0" upper="1.2" velocity="3.0"/>
-    </joint>
-    <!-- dedo opuesto (mimic) -->
-    <joint name="gripper_right" type="revolute">
-      <origin xyz="0.0 -0.018 0.01" rpy="0 0 0"/>
-      <parent link="gripper_base"/>
-      <child link="gripper_finger_right"/>
-      <axis xyz="1 0 0"/>
-      <limit effort="5.0" lower="-1.2" upper="0.0" velocity="3.0"/>
+      <parent link="${parent}"/><child link="gripper_finger_right"/>
+      <axis xyz="0 1 0"/>
+      <limit effort="5.0" lower="-0.6" upper="0.0" velocity="2.0"/>
       <mimic joint="gripper" multiplier="-1.0"/>
     </joint>
-  </xacro:macro>
-  <xacro:macro name="gripper_finger_primitive" params="side reflect">
-    <link name="gripper_finger_${side}">
-      <inertial>
-        <mass value="0.01"/>
-        <inertia ixx="1e-6" ixy="0" ixz="0" iyy="1e-6" iyz="0" izz="1e-6"/>
-      </inertial>
+    <link name="gripper_finger_right">
+      <inertial><mass value="0.01"/>
+        <inertia ixx="1e-6" ixy="0" ixz="0" iyy="1e-6" iyz="0" izz="1e-6"/></inertial>
       <visual>
-        <origin xyz="0 ${reflect*0.004} 0.02" rpy="0 0 0"/>
-        <geometry><box size="0.008 0.008 0.04"/></geometry>
+        <origin xyz="-0.012 0 0.018" rpy="0 0 0"/>
+        <geometry><box size="0.006 0.012 0.036"/></geometry>
         <material name="red"/>
       </visual>
-      <collision>
-        <origin xyz="0 ${reflect*0.004} 0.02" rpy="0 0 0"/>
-        <geometry><box size="0.008 0.008 0.04"/></geometry>
-      </collision>
     </link>
   </xacro:macro>
-  <!-- ===== MESHES ===== -->
-  <!-- Dedos con los STL reales (rescatados de twin_ws). El offset replica la
-       compensacion de marco global usada en twin (z negativo). Afinar en RViz. -->
-  <xacro:macro name="gripper_mesh" params="parent *origin grip_z:=-0.37">
-    <joint name="gripper" type="revolute">
-      <xacro:insert_block name="origin"/>
-      <parent link="${parent}"/>
-      <child link="gripper_finger_left"/>
-      <axis xyz="1 0 0"/>
-      <limit effort="5.0" lower="-0.13" upper="1.2" velocity="3.0"/>
+  <!-- ===== MESH FUSIONADO (fijo) ===== -->
+  <!-- Une el gripper real al eslabón de la muñeca como UN solo cuerpo rígido.
+       grip_z desplaza la malla (marco CAD global de twin); afínalo en RViz. -->
+  <xacro:macro name="gripper_mesh_fused" params="parent grip_z:=-0.36">
+    <joint name="gripper_fixed" type="fixed">
+      <origin xyz="0 0 0" rpy="0 0 0"/>
+      <parent link="${parent}"/><child link="gripper_link"/>
     </joint>
-    <link name="gripper_finger_left">
-      <inertial>
-        <mass value="0.02"/>
-        <inertia ixx="1e-5" ixy="0" ixz="0" iyy="1e-5" iyz="0" izz="1e-5"/>
-      </inertial>
+    <link name="gripper_link">
+      <inertial><mass value="0.04"/>
+        <inertia ixx="2e-5" ixy="0" ixz="0" iyy="2e-5" iyz="0" izz="2e-5"/></inertial>
       <visual>
         <origin xyz="0.0 0.008 ${grip_z}" rpy="0 0 0"/>
@@ -95,25 +62,4 @@
         <material name="black"/>
       </visual>
-      <collision>
-        <origin xyz="0.0 0.008 ${grip_z}" rpy="0 0 0"/>
-        <geometry>
-          <mesh filename="package://robotfun_description/meshes/gripper/left_gripper.stl"
-                scale="0.001 0.001 0.001"/>
-        </geometry>
-      </collision>
-    </link>
-    <joint name="gripper_right" type="revolute">
-      <origin xyz="0 0 0" rpy="0 0 0"/>
-      <parent link="${parent}"/>
-      <child link="gripper_finger_right"/>
-      <axis xyz="1 0 0"/>
-      <limit effort="5.0" lower="-1.2" upper="0.13" velocity="3.0"/>
-      <mimic joint="gripper" multiplier="-1.0"/>
-    </joint>
-    <link name="gripper_finger_right">
-      <inertial>
-        <mass value="0.02"/>
-        <inertia ixx="1e-5" ixy="0" ixz="0" iyy="1e-5" iyz="0" izz="1e-5"/>
-      </inertial>
       <visual>
         <origin xyz="0.0 -0.008 ${grip_z}" rpy="0 0 0"/>
@@ -124,11 +70,4 @@
         <material name="black"/>
       </visual>
-      <collision>
-        <origin xyz="0.0 -0.008 ${grip_z}" rpy="0 0 0"/>
-        <geometry>
-          <mesh filename="package://robotfun_description/meshes/gripper/right_gripper.stl"
-                scale="0.001 0.001 0.001"/>
-        </geometry>
-      </collision>
     </link>
   </xacro:macro>

File: src/robotfun_description/urdf/robotfun.urdf.xacro (robot description, xacro)
@@ -3,10 +3,8 @@
      robotfun.urdf.xacro  —  MODELO DE MEDIDAS REALES (primitivas)
      ===========================================================================
-     Brazo 4 GDL (yaw + 3 pitch) + gripper, dibujado con PRIMITIVAS dimensionadas
-     a las medidas reales del robot. Comparte el esqueleto (juntas joint_1..joint_4)
-     con el modelo de meshes, y reproduce EXACTAMENTE la FK del núcleo
-     `robotfun_kinematics` (TF == FK). Es el modelo para VERIFICAR la cinemática
-     inversa. Incluye inertiales (preparado para Gazebo/MoveIt2).
-     Para ver las piezas reales del CAD:  display.launch.py model:=meshes
+     Brazo 4 GDL RECTO + gripper, con PRIMITIVAS dimensionadas a las medidas
+     reales (D1=0.1375 A2=0.1277 A3=0.125 HAND=0.12). Reproduce EXACTAMENTE la FK
+     del núcleo (TF == FK). Es el modelo para VERIFICAR el DH y la cinemática
+     inversa. Para ver las piezas reales:  display.launch.py model:=meshes
      ========================================================================== -->
 <robot name="robotfun" xmlns:xacro="http://www.ros.org/wiki/xacro">
@@ -15,6 +13,7 @@
   <xacro:include filename="$(find robotfun_description)/urdf/common/gripper.macro.xacro"/>
   <xacro:robotfun_arm use_mesh="false"/>
-  <xacro:gripper_primitive parent="tool0">
-    <origin xyz="0 0 0.006" rpy="0 0 0"/>
+  <!-- gripper de prueba (móvil) en la zona de la mano -->
+  <xacro:gripper_primitive parent="link_4">
+    <origin xyz="0 0 0.084" rpy="0 0 0"/>
   </xacro:gripper_primitive>
 </robot>

File: src/robotfun_description/urdf/robotfun_meshes.urdf.xacro (robot description, xacro)
@@ -4,13 +4,13 @@
      ===========================================================================
      Mismo esqueleto y MISMAS juntas (joint_1..joint_4) que el modelo de medidas
-     reales, pero con las PIEZAS REALES del robot (meshes de brazo_ws, ya limpio:
-     sin engranajes ni eslabón sobrante, escala uniforme 0.001). Sirve para ver
-     el robot tal cual es y comparar con el modelo primitivo (ambos se mueven
-     idéntico, los mueve el mismo /joint_states). Se monta el GRIPPER real
-     rescatado de twin_ws.
-     CENTRADO de meshes: las STL vienen en un marco CAD global; el <visual> de
-     cada link compensa la traslación. Si alguna pieza se ve descentrada en XY,
-     ajusta su <origin> (ver scripts/mesh_bbox.py). El modelo primitivo es la
-     referencia cinemática exacta.
+     reales, pero con las PIEZAS REALES (meshes de brazo_ws). El gripper real
+     (twin_ws) se FUSIONA a link_4 (la muñeca/soporte) como un solo cuerpo: ya no
+     hay cubo ni piezas flotando.
+     Se mueve con el mismo /joint_states que el modelo primitivo ⇒ cuando mandas
+     una pose a la IK, este modelo de hardware también se mueve.
+     CENTRADO: las STL vienen en un marco CAD global; el <origin> de cada <visual>
+     (en arm.macro.xacro) y el grip_z del gripper son el punto de partida. Si algo
+     se ve desfasado, ajústalo en RViz (ver scripts/mesh_bbox.py). El modelo
+     primitivo (model:=primitives) es la referencia cinemática exacta.
      ========================================================================== -->
 <robot name="robotfun_meshes" xmlns:xacro="http://www.ros.org/wiki/xacro">
@@ -19,8 +19,5 @@
   <xacro:include filename="$(find robotfun_description)/urdf/common/gripper.macro.xacro"/>
   <xacro:robotfun_arm use_mesh="true"/>
-  <!-- Gripper real (twin_ws) en el TCP. El offset es punto de partida: afínalo
-       en RViz si hace falta (ver README). -->
-  <xacro:gripper_mesh parent="tool0" grip_z="-0.03">
-    <origin xyz="0 0 0.0" rpy="0 0 0"/>
-  </xacro:gripper_mesh>
+  <!-- gripper real fusionado a la muñeca (un solo eslabón). Afina grip_z en RViz. -->
+  <xacro:gripper_mesh_fused parent="link_4" grip_z="-0.36"/>
 </robot>
