Commit message: Aplicar tabla DH del usuario (L0..L5) y limpiar el modelo de meshes
Medidas según la tabla DH del usuario (brazo_ws actualizado):
  L0=0.010 (offset radial base), L1=0.063, L2=0.120, A3=L3+L4=0.120, HAND=L5=0.11.
  FK(HOME) → TCP=[0.010, 0, 0.413]. La IK analítica considera el offset de hombro
  L0. Restricción articular −90/0/+90 (HOME=0 ⇒ servo a 90°).

- Modelo PRIMITIVO (model:=primitives): esqueleto de la tabla DH, reproduce
  EXACTAMENTE la FK (TF==FK a 1e-16). Es la referencia para verificar la IK.
- Modelo de MESHES (model:=meshes): standalone con los orígenes del CAD
  (brazo.urdf, donde las mallas se alinean), mismas juntas joint_1..joint_4 y
  sentidos de giro (axis 0 -1 0). eslabon3 re-exportado (escala 0.001 uniforme).
  SIN cubo y SIN el gripper flotante de twin (eliminados). tool0 = solo frame.
- Núcleo/tests/docs/scripts actualizados; mallas re-importadas desde brazo_ws.

Co-Authored-By: Claude Opus 4.8 <noreply@anthropic.com>
Claude-Session: https://claude.ai/code/session_01HQm53DmrqYUT2G9sJ8qfUh

File: src/robotfun_description/urdf/common/arm.macro.xacro (robot description, xacro)
@@ -1,131 +1,91 @@
 <?xml version="1.0"?>
 <!-- ============================================================================
-     arm.macro.xacro  —  esqueleto compartido del brazo 4 GDL (RECTO)
+     arm.macro.xacro  —  esqueleto PRIMITIVO (tabla DH del usuario)
      ===========================================================================
-     Cadena base_link → link_1..link_4 → tool0 con las medidas reales y el brazo
-     RECTO (sin offsets). Reproduce EXACTAMENTE la FK del núcleo (TF == FK a 1e-16).
-         D1=0.1375  A2=0.1277  A3=0.125 (medido)  HAND=0.12 (medido)  [m]
-     El mismo esqueleto sirve para los dos modelos:
-        use_mesh=false → PRIMITIVAS dimensionadas a las medidas (verifica DH/IK).
-        use_mesh=true  → PIEZAS REALES del CAD (visualización del hardware).
-     Ejes: joint_1=(0 0 1) yaw; joint_2/3/4=(0 -1 0) pitch. tool0 es solo un frame
-     (sin cubo). El gripper se añade aparte (gripper.macro.xacro).
+     Brazo 4 GDL RECTO dibujado con PRIMITIVAS dimensionadas a la tabla DH:
+         L0=0.010 (offset base)  L1=0.063  L2=0.120  A3=0.120  HAND=0.11  [m]
+     Reproduce EXACTAMENTE la FK del núcleo (TF == FK). Es el modelo para
+     VERIFICAR el DH y la cinemática inversa.  FK(HOME) → TCP=[0.010, 0, 0.413].
+     Ejes: joint_1=(0 0 1) yaw; joint_2/3/4=(0 -1 0) pitch. tool0 = frame (sin cubo).
      ========================================================================== -->
 <robot xmlns:xacro="http://www.ros.org/wiki/xacro">
-  <xacro:property name="mesh" value="package://robotfun_description/meshes/arm"/>
-  <xacro:property name="lo" value="-1.5708"/>   <!-- −90°, límite real del servo -->
-  <xacro:property name="hi" value="1.5708"/>    <!-- +90° (HOME=0 ⇒ servo a 90°) -->
-  <xacro:macro name="robotfun_arm" params="use_mesh:=false">
+  <xacro:property name="lo" value="-1.5708"/>   <!-- −90° (HOME=0 ⇒ servo a 90°) -->
+  <xacro:property name="hi" value="1.5708"/>    <!-- +90° -->
+  <xacro:macro name="robotfun_arm">
     <link name="world"/>
     <joint name="base_joint" type="fixed">
       <origin xyz="0 0 0" rpy="0 0 0"/><parent link="world"/><child link="base_link"/>
     </joint>
-    <!-- ===== base_link ===== -->
+    <!-- base_link (soporte fijo) -->
     <link name="base_link">
       <inertial><mass value="1.0"/>
         <inertia ixx="0.01" ixy="0" ixz="0" iyy="0.01" iyz="0" izz="0.01"/></inertial>
       <visual>
-        <xacro:if value="${use_mesh}">
-          <origin xyz="0 0 0" rpy="0 0 0"/>
-          <geometry><mesh filename="${mesh}/base_link.stl" scale="0.001 0.001 0.001"/></geometry>
-          <material name="grey"/>
-        </xacro:if>
-        <xacro:unless value="${use_mesh}">
-          <origin xyz="0 0 0.0309" rpy="0 0 0"/>
-          <geometry><cylinder radius="0.045" length="0.0617"/></geometry>
-          <material name="grey"/>
-        </xacro:unless>
+        <origin xyz="0 0 0.015" rpy="0 0 0"/>
+        <geometry><cylinder radius="0.045" length="0.03"/></geometry>
+        <material name="grey"/>
       </visual>
     </link>
+    <!-- joint_1 yaw (en la base) -->
     <joint name="joint_1" type="revolute">
-      <origin xyz="0 0 0.0617" rpy="0 0 0"/><parent link="base_link"/><child link="link_1"/>
+      <origin xyz="0 0 0" rpy="0 0 0"/><parent link="base_link"/><child link="link_1"/>
       <axis xyz="0 0 1"/><limit lower="${lo}" upper="${hi}" effort="10.0" velocity="1.5"/>
     </joint>
-    <!-- ===== link_1 (yaw → hombro) ===== -->
+    <!-- link_1: columna de yaw hasta el hombro (L0 radial, L1 alto) -->
     <link name="link_1">
-      <inertial><origin xyz="0 0 0.038"/><mass value="0.5"/>
+      <inertial><origin xyz="0.005 0 0.032"/><mass value="0.5"/>
         <inertia ixx="1e-3" ixy="0" ixz="0" iyy="1e-3" iyz="0" izz="1e-3"/></inertial>
       <visual>
-        <xacro:if value="${use_mesh}">
-          <origin xyz="0 0 -0.0617" rpy="0 0 0"/>
-          <geometry><mesh filename="${mesh}/eslabon1_link.stl" scale="0.001 0.001 0.001"/></geometry>
-          <material name="white_grey"/>
-        </xacro:if>
-        <xacro:unless value="${use_mesh}">
-          <origin xyz="0 0 0.0379" rpy="0 0 0"/>
-          <geometry><cylinder radius="0.022" length="0.0758"/></geometry>
-          <material name="black"/>
-        </xacro:unless>
+        <origin xyz="0.005 0 0.032" rpy="0 0.156 0"/>
+        <geometry><cylinder radius="0.022" length="0.064"/></geometry>
+        <material name="black"/>
       </visual>
     </link>
+    <!-- joint_2 hombro: offset radial L0=0.010, alto L1=0.063 -->
     <joint name="joint_2" type="revolute">
-      <origin xyz="0 0 0.0758" rpy="0 0 0"/><parent link="link_1"/><child link="link_2"/>
+      <origin xyz="0.010 0 0.063" rpy="0 0 0"/><parent link="link_1"/><child link="link_2"/>
       <axis xyz="0 -1 0"/><limit lower="${lo}" upper="${hi}" effort="10.0" velocity="1.5"/>
     </joint>
-    <!-- ===== link_2 (brazo, A2) ===== -->
+    <!-- link_2: brazo L2=0.120 -->
     <link name="link_2">
-      <inertial><origin xyz="0 0 0.064"/><mass value="0.4"/>
+      <inertial><origin xyz="0 0 0.06"/><mass value="0.4"/>
         <inertia ixx="1e-3" ixy="0" ixz="0" iyy="1e-3" iyz="0" izz="1e-3"/></inertial>
       <visual>
-        <xacro:if value="${use_mesh}">
-          <origin xyz="0 0 -0.1375" rpy="0 0 0"/>
-          <geometry><mesh filename="${mesh}/eslabon2_link.stl" scale="0.001 0.001 0.001"/></geometry>
-          <material name="white_grey"/>
-        </xacro:if>
-        <xacro:unless value="${use_mesh}">
-          <origin xyz="0 0 0.0639" rpy="0 0 0"/>
-          <geometry><cylinder radius="0.018" length="0.1277"/></geometry>
-          <material name="red"/>
-        </xacro:unless>
+        <origin xyz="0 0 0.060" rpy="0 0 0"/>
+        <geometry><cylinder radius="0.018" length="0.120"/></geometry>
+        <material name="red"/>
       </visual>
     </link>
     <joint name="joint_3" type="revolute">
-      <origin xyz="0 0 0.1277" rpy="0 0 0"/><parent link="link_2"/><child link="link_3"/>
+      <origin xyz="0 0 0.120" rpy="0 0 0"/><parent link="link_2"/><child link="link_3"/>
       <axis xyz="0 -1 0"/><limit lower="${lo}" upper="${hi}" effort="10.0" velocity="1.5"/>
     </joint>
-    <!-- ===== link_3 (antebrazo, A3=0.125) ===== -->
+    <!-- link_3: antebrazo A3=0.120 -->
     <link name="link_3">
-      <inertial><origin xyz="0 0 0.0625"/><mass value="0.3"/>
+      <inertial><origin xyz="0 0 0.06"/><mass value="0.3"/>
         <inertia ixx="8e-4" ixy="0" ixz="0" iyy="8e-4" iyz="0" izz="8e-4"/></inertial>
       <visual>
-        <xacro:if value="${use_mesh}">
-          <!-- eslabon3 se exportó en otra escala: usa 0.0001 (a 0.001 flota a ~2.4 m). -->
-          <origin xyz="0 0 -0.2652" rpy="0 0 0"/>
-          <geometry><mesh filename="${mesh}/eslabon3_link.stl" scale="0.0001 0.0001 0.0001"/></geometry>
-          <material name="white_grey"/>
-        </xacro:if>
-        <xacro:unless value="${use_mesh}">
-          <origin xyz="0 0 0.0625" rpy="0 0 0"/>
-          <geometry><cylinder radius="0.015" length="0.125"/></geometry>
-          <material name="blue"/>
-        </xacro:unless>
+        <origin xyz="0 0 0.060" rpy="0 0 0"/>
+        <geometry><cylinder radius="0.015" length="0.120"/></geometry>
+        <material name="blue"/>
       </visual>
     </link>
     <joint name="joint_4" type="revolute">
-      <origin xyz="0 0 0.125" rpy="0 0 0"/><parent link="link_3"/><child link="link_4"/>
+      <origin xyz="0 0 0.120" rpy="0 0 0"/><parent link="link_3"/><child link="link_4"/>
       <axis xyz="0 -1 0"/><limit lower="${lo}" upper="${hi}" effort="10.0" velocity="1.5"/>
     </joint>
-    <!-- ===== link_4 (muñeca + base del gripper = UN solo eslabón) =====
-         En el modelo de meshes, link_4 = eslabon4 (pieza de muñeca/soporte del
-         gripper). El gripper se fusiona aquí mismo (gripper.macro.xacro). -->
+    <!-- link_4: mano HAND=0.11 (muñeca → punta) -->
     <link name="link_4">
-      <inertial><origin xyz="0 0 0.06"/><mass value="0.2"/>
+      <inertial><origin xyz="0 0 0.055"/><mass value="0.2"/>
         <inertia ixx="5e-4" ixy="0" ixz="0" iyy="5e-4" iyz="0" izz="5e-4"/></inertial>
       <visual>
-        <xacro:if value="${use_mesh}">
-          <origin xyz="0 0 -0.3902" rpy="0 0 0"/>
-          <geometry><mesh filename="${mesh}/eslabon4_link.stl" scale="0.001 0.001 0.001"/></geometry>
-          <material name="black"/>
-        </xacro:if>
-        <xacro:unless value="${use_mesh}">
-          <origin xyz="0 0 0.06" rpy="0 0 0"/>
-          <geometry><cylinder radius="0.013" length="0.12"/></geometry>
-          <material name="black"/>
-        </xacro:unless>
+        <origin xyz="0 0 0.055" rpy="0 0 0"/>
+        <geometry><cylinder radius="0.013" length="0.110"/></geometry>
+        <material name="black"/>
       </visual>
     </link>
-    <!-- tool0 = TCP (punta del gripper, HAND=0.12). Solo FRAME, sin cubo. -->
+    <!-- tool0 = TCP (punta del gripper). Solo frame, sin cubo. -->
     <joint name="tool_fixed" type="fixed">
-      <origin xyz="0 0 0.12" rpy="0 0 0"/><parent link="link_4"/><child link="tool0"/>
+      <origin xyz="0 0 0.110" rpy="0 0 0"/><parent link="link_4"/><child link="tool0"/>
     </joint>
     <link name="tool0"/>

File: src/robotfun_description/urdf/common/gripper.macro.xacro (robot description, xacro)
@@ -43,32 +43,3 @@
     </link>
   </xacro:macro>
-  <!-- ===== MESH FUSIONADO (fijo) ===== -->
-  <!-- Une el gripper real al eslabón de la muñeca como UN solo cuerpo rígido.
-       grip_z desplaza la malla (marco CAD global de twin); afínalo en RViz. -->
-  <xacro:macro name="gripper_mesh_fused" params="parent grip_z:=-0.36">
-    <joint name="gripper_fixed" type="fixed">
-      <origin xyz="0 0 0" rpy="0 0 0"/>
-      <parent link="${parent}"/><child link="gripper_link"/>
-    </joint>
-    <link name="gripper_link">
-      <inertial><mass value="0.04"/>
-        <inertia ixx="2e-5" ixy="0" ixz="0" iyy="2e-5" iyz="0" izz="2e-5"/></inertial>
-      <visual>
-        <origin xyz="0.0 0.008 ${grip_z}" rpy="0 0 0"/>
-        <geometry>
-          <mesh filename="package://robotfun_description/meshes/gripper/left_gripper.stl"
-                scale="0.001 0.001 0.001"/>
-        </geometry>
-        <material name="black"/>
-      </visual>
-      <visual>
-        <origin xyz="0.0 -0.008 ${grip_z}" rpy="0 0 0"/>
-        <geometry>
-          <mesh filename="package://robotfun_description/meshes/gripper/right_gripper.stl"
-                scale="0.001 0.001 0.001"/>
-        </geometry>
-        <material name="black"/>
-      </visual>
-    </link>
-  </xacro:macro>
 </robot>

File: src/robotfun_description/urdf/robotfun.urdf.xacro (robot description, xacro)
@@ -1,10 +1,10 @@
 <?xml version="1.0"?>
 <!-- ============================================================================
-     robotfun.urdf.xacro  —  MODELO DE MEDIDAS REALES (primitivas)
+     robotfun.urdf.xacro  —  MODELO DE MEDIDAS REALES (primitivas, tabla DH)
      ===========================================================================
-     Brazo 4 GDL RECTO + gripper, con PRIMITIVAS dimensionadas a las medidas
-     reales (D1=0.1375 A2=0.1277 A3=0.125 HAND=0.12). Reproduce EXACTAMENTE la FK
+     Brazo 4 GDL RECTO + gripper, con PRIMITIVAS a las medidas de tu tabla DH
+     (L0=0.010 L1=0.063 L2=0.120 A3=0.120 HAND=0.11). Reproduce EXACTAMENTE la FK
      del núcleo (TF == FK). Es el modelo para VERIFICAR el DH y la cinemática
-     inversa. Para ver las piezas reales:  display.launch.py model:=meshes
+     inversa. Para ver tus piezas reales:  display.launch.py model:=meshes
      ========================================================================== -->
 <robot name="robotfun" xmlns:xacro="http://www.ros.org/wiki/xacro">
@@ -12,8 +12,8 @@
   <xacro:include filename="$(find robotfun_description)/urdf/common/arm.macro.xacro"/>
   <xacro:include filename="$(find robotfun_description)/urdf/common/gripper.macro.xacro"/>
-  <xacro:robotfun_arm use_mesh="false"/>
+  <xacro:robotfun_arm/>
   <!-- gripper de prueba (móvil) en la zona de la mano -->
   <xacro:gripper_primitive parent="link_4">
-    <origin xyz="0 0 0.084" rpy="0 0 0"/>
+    <origin xyz="0 0 0.078" rpy="0 0 0"/>
   </xacro:gripper_primitive>
 </robot>

File: src/robotfun_description/urdf/robotfun_meshes.urdf.xacro (robot description, xacro)
@@ -3,21 +3,84 @@
      robotfun_meshes.urdf.xacro  —  MODELO DE PIEZAS REALES (meshes del CAD)
      ===========================================================================
-     Mismo esqueleto y MISMAS juntas (joint_1..joint_4) que el modelo de medidas
-     reales, pero con las PIEZAS REALES (meshes de brazo_ws). El gripper real
-     (twin_ws) se FUSIONA a link_4 (la muñeca/soporte) como un solo cuerpo: ya no
-     hay cubo ni piezas flotando.
-     Se mueve con el mismo /joint_states que el modelo primitivo ⇒ cuando mandas
-     una pose a la IK, este modelo de hardware también se mueve.
-     CENTRADO: las STL vienen en un marco CAD global; el <origin> de cada <visual>
-     (en arm.macro.xacro) y el grip_z del gripper son el punto de partida. Si algo
-     se ve desfasado, ajústalo en RViz (ver scripts/mesh_bbox.py). El modelo
-     primitivo (model:=primitives) es la referencia cinemática exacta.
+     Visualización del robot real con TUS piezas (meshes de brazo_ws, ya con
+     eslabon3 re-exportado y piezas unidas). Usa los orígenes de tu brazo.urdf
+     (donde las mallas están alineadas) y MISMAS juntas (joint_1..joint_4) que el
+     modelo primitivo, con los pitch en axis="0 -1 0" para que se muevan en el
+     mismo sentido. Lo mueve el mismo /joint_states ⇒ cuando mandas una pose a la
+     IK, este modelo de hardware también se mueve.
+     Limpieza: SIN cubo y SIN el gripper flotante de twin (eliminado). El gripper
+     real es parte de eslabon4 (piezas unidas). tool0 es solo un frame.
+     Nota: las proporciones vienen de tu brazo.urdf (CAD). El modelo PRIMITIVO
+     (model:=primitives) es la referencia exacta de la tabla DH para verificar la
+     cinemática. Si quieres que las mallas coincidan 1:1 con la DH, habría que
+     re-exportarlas a las longitudes L1..L5.
      ========================================================================== -->
 <robot name="robotfun_meshes" xmlns:xacro="http://www.ros.org/wiki/xacro">
   <xacro:include filename="$(find robotfun_description)/urdf/common/materials.xacro"/>
-  <xacro:include filename="$(find robotfun_description)/urdf/common/arm.macro.xacro"/>
-  <xacro:include filename="$(find robotfun_description)/urdf/common/gripper.macro.xacro"/>
-  <xacro:robotfun_arm use_mesh="true"/>
-  <!-- gripper real fusionado a la muñeca (un solo eslabón). Afina grip_z en RViz. -->
-  <xacro:gripper_mesh_fused parent="link_4" grip_z="-0.36"/>
+  <xacro:property name="mesh" value="package://robotfun_description/meshes/arm"/>
+  <xacro:property name="lo" value="-1.5708"/>
+  <xacro:property name="hi" value="1.5708"/>
+  <link name="world"/>
+  <joint name="base_joint" type="fixed">
+    <origin xyz="0 0 0" rpy="0 0 0"/><parent link="world"/><child link="base_link"/>
+  </joint>
+  <link name="base_link">
+    <inertial><mass value="1.0"/>
+      <inertia ixx="0.01" ixy="0" ixz="0" iyy="0.01" iyz="0" izz="0.01"/></inertial>
+    <visual>
+      <origin xyz="0 0 0" rpy="0 0 0"/>
+      <geometry><mesh filename="${mesh}/base_link.stl" scale="0.001 0.001 0.001"/></geometry>
+      <material name="grey"/>
+    </visual>
+  </link>
+  <joint name="joint_1" type="revolute">
+    <origin xyz="0 0 0.0617" rpy="0 0 0"/><parent link="base_link"/><child link="link_1"/>
+    <axis xyz="0 0 1"/><limit lower="${lo}" upper="${hi}" effort="10.0" velocity="1.5"/>
+  </joint>
+  <link name="link_1">
+    <visual>
+      <origin xyz="0 0 -0.0617" rpy="0 0 0"/>
+      <geometry><mesh filename="${mesh}/eslabon1_link.stl" scale="0.001 0.001 0.001"/></geometry>
+      <material name="white_grey"/>
+    </visual>
+  </link>
+  <joint name="joint_2" type="revolute">
+    <origin xyz="0 0 0.0758" rpy="0 0 0"/><parent link="link_1"/><child link="link_2"/>
+    <axis xyz="0 -1 0"/><limit lower="${lo}" upper="${hi}" effort="10.0" velocity="1.5"/>
+  </joint>
+  <link name="link_2">
+    <visual>
+      <origin xyz="0 0 -0.1375" rpy="0 0 0"/>
+      <geometry><mesh filename="${mesh}/eslabon2_link.stl" scale="0.001 0.001 0.001"/></geometry>
+      <material name="white_grey"/>
+    </visual>
+  </link>
+  <joint name="joint_3" type="revolute">
+    <origin xyz="0 0 0.1277" rpy="0 0 0"/><parent link="link_2"/><child link="link_3"/>
+    <axis xyz="0 -1 0"/><limit lower="${lo}" upper="${hi}" effort="10.0" velocity="1.5"/>
+  </joint>
+  <link name="link_3">
+    <visual>
+      <origin xyz="0 0 -0.2652" rpy="0 0 0"/>
+      <geometry><mesh filename="${mesh}/eslabon3_link.stl" scale="0.001 0.001 0.001"/></geometry>
+      <material name="white_grey"/>
+    </visual>
+  </link>
+  <joint name="joint_4" type="revolute">
+    <origin xyz="0.038 0 0.1213" rpy="0 0 0"/><parent link="link_3"/><child link="link_4"/>
+    <axis xyz="0 -1 0"/><limit lower="${lo}" upper="${hi}" effort="10.0" velocity="1.5"/>
+  </joint>
+  <!-- link_4 = eslabon4 (muñeca + gripper unidos: un solo eslabón) -->
+  <link name="link_4">
+    <visual>
+      <origin xyz="-0.038 0 -0.3865" rpy="0 0 0"/>
+      <geometry><mesh filename="${mesh}/eslabon4_link.stl" scale="0.001 0.001 0.001"/></geometry>
+      <material name="black"/>
+    </visual>
+  </link>
+  <!-- tool0 = TCP (punta del gripper, HAND≈0.11). Solo frame. -->
+  <joint name="tool_fixed" type="fixed">
+    <origin xyz="0 0 0.11" rpy="0 0 0"/><parent link="link_4"/><child link="tool0"/>
+  </joint>
+  <link name="tool0"/>
 </robot>
