Commit message: Reestructura a 5 actuadores joint_1..joint_5 (joint_5 = gripper) + reasigna pines
Reorganiza el proyecto como si el robot siempre hubiese tenido 5 actuadores
(sin el antiguo roll de muñeca): joint_4 = pitch de muñeca, joint_5 = gripper.

Firmware (robotfun_esp32_microros.ino):
- joint_name_buf / JOINT_LABEL = joint_1..joint_5 (gripper renombrado a joint_5).
- Reasigna pines tras quitar el roll: POT revive 35 (joint_4), continúa 27
  (gripper) y anula 26 -> {32,33,34,35,27}; SERVO revive 18, continúa 19 y
  anula 21 -> {2,4,5,18,19}. Documenta que solo los pines de pot fueron fijados
  explícitamente por el usuario.
- Elimina el servo muerto de roll (DEAD_ROLL_PIN) y su bloque; ya no existe.
- Conserva la calibración: RAW_ZERO={1267,1232,1265,1405,1302},
  FEEDBACK_DIRECTION={1,1,-1,-1,1}, SERVO_DIRECTION={1,-1,1,-1,1}.
- Corrige el rango del gripper (joint_5) a [0,70] grados.

Sketch de calibración (robotfun_calibracion_raw.ino): POT {32,33,34,35,27},
etiquetas joint_1..joint_5.

Cinemática: GRIPPER_JOINT_NAME = "joint_5"; trajectory_node usa la constante
en vez del literal "gripper".

Descripción: gripper.macro.xacro renombra el joint actuado a "joint_5" (mimic
joint_5_right -> joint_5); joint_limits.yaml e initial_positions.yaml usan joint_5.

Docs (ARCHITECTURE, ROADMAP, README firmware y raíz): interfaz joint_1..joint_5,
roll eliminado por completo y tabla de pines reasignada.

Verificado: FK(HOME) TCP=[0.010,0,0.413]; TF==FK a 2e-17; 9/9 tests; xacro OK.

Co-Authored-By: Claude Opus 4.8 <noreply@anthropic.com>
Claude-Session: https://claude.ai/code/session_01HQm53DmrqYUT2G9sJ8qfUh

File: src/robotfun_description/urdf/common/gripper.macro.xacro (robot description, xacro)
@@ -2,14 +2,12 @@
 <!-- ============================================================================
      gripper.macro.xacro
-     Dos macros, sin el cubo anterior:
-       * gripper_primitive : gripper de 1 GDL (canal 6) con dedos finos de caja;
-         se mueve (joint "gripper") para el modelo de medidas reales.
-       * gripper_mesh_fused: el gripper real (STL de twin_ws) FUSIONADO y FIJO al
-         eslabón de la muñeca → "un solo eslabón" con link_4. Sin cubo, sin flotar.
+       * gripper_primitive : gripper de 1 GDL con dedos finos de caja; se mueve con
+         el joint "joint_5" (el 5º actuador, físicamente el gripper) para el modelo
+         de medidas reales. Sin el cubo anterior.
      ========================================================================== -->
 <robot xmlns:xacro="http://www.ros.org/wiki/xacro">
   <!-- ===== PRIMITIVO (móvil) ===== -->
   <xacro:macro name="gripper_primitive" params="parent *origin">
-    <joint name="gripper" type="revolute">
+    <joint name="joint_5" type="revolute">
       <xacro:insert_block name="origin"/>
       <parent link="${parent}"/><child link="gripper_finger_left"/>
@@ -26,10 +24,10 @@
       </visual>
     </link>
-    <joint name="gripper_right" type="revolute">
+    <joint name="joint_5_right" type="revolute">
       <xacro:insert_block name="origin"/>
       <parent link="${parent}"/><child link="gripper_finger_right"/>
       <axis xyz="0 1 0"/>
       <limit effort="5.0" lower="-0.6" upper="0.0" velocity="2.0"/>
-      <mimic joint="gripper" multiplier="-1.0"/>
+      <mimic joint="joint_5" multiplier="-1.0"/>
     </joint>
     <link name="gripper_finger_right">

Commit message: URDF: amplia limite del gripper (joint_5) a 0..1.22 rad para RViz
El comando abre el gripper a 0.70 rad pero el URDF lo topaba a 0.6 -> RViz
recortaba el dedo. Se amplia joint_5 a [0, 1.22] y su mimic joint_5_right a
[-1.22, 0], igual que el rango del firmware (0..70 grados) y joint_limits.yaml.
Asi RViz refleja el gripper completo al sincronizar con el pick & place.

Co-Authored-By: Claude Opus 4.8 <noreply@anthropic.com>
Claude-Session: https://claude.ai/code/session_01HQm53DmrqYUT2G9sJ8qfUh

File: src/robotfun_description/urdf/common/gripper.macro.xacro (robot description, xacro)
@@ -13,5 +13,6 @@
       <parent link="${parent}"/><child link="gripper_finger_left"/>
       <axis xyz="0 1 0"/>
-      <limit effort="5.0" lower="0.0" upper="0.6" velocity="2.0"/>
+      <!-- rango 0..70° (1.22 rad), igual que el firmware/command; asi RViz no recorta -->
+      <limit effort="5.0" lower="0.0" upper="1.22" velocity="2.0"/>
     </joint>
     <link name="gripper_finger_left">
@@ -28,5 +29,5 @@
       <parent link="${parent}"/><child link="gripper_finger_right"/>
       <axis xyz="0 1 0"/>
-      <limit effort="5.0" lower="-0.6" upper="0.0" velocity="2.0"/>
+      <limit effort="5.0" lower="-1.22" upper="0.0" velocity="2.0"/>
       <mimic joint="joint_5" multiplier="-1.0"/>
     </joint>
